Commit message: Changed names to English

File: wezelROS/description/urdf/gripper.urdf (robot description, URDF)
Before this commit: robot chwytak, 7 links, 6 joints
Links:
- removed link palec1
- removed link palec1_obrot
- removed link palec2
- removed link palec2_obrot
- removed link palec3
- removed link palec3_obrot
- added link finger_link1; visual mesh filename=package://wezelROS/description/meshes/finger.stl
- added link finger_link2; visual mesh filename=package://wezelROS/description/meshes/finger.stl
- added link finger_link3; visual mesh filename=package://wezelROS/description/meshes/finger.stl
- added link rotator_link1; visual mesh filename=package://wezelROS/description/meshes/finger_rotator.stl
- added link rotator_link2; visual mesh filename=package://wezelROS/description/meshes/finger_rotator.stl
- added link rotator_link3; visual mesh filename=package://wezelROS/description/meshes/finger_rotator.stl
Joints:
- removed joint swivel1
- removed joint swivel2
- removed joint swivel3
- removed joint swivelpalec
- removed joint swivelpalec2
- removed joint swivelpalec3
- added joint finger1: type revolute, parent rotator_link1, child finger_link1, origin xyz=0 0 0, axis 1 0 0, limit lower=-1 upper=1.57 effort=30 velocity=5
- added joint finger2: type revolute, parent rotator_link2, child finger_link2, origin xyz=0 0 0, axis 1 0 0, limit lower=-1.57 upper=1 effort=30 velocity=5
- added joint finger3: type revolute, parent rotator_link3, child finger_link3, origin xyz=0 0 0, axis 1 0 0, limit lower=-1.57 upper=1 effort=30 velocity=5
- added joint rotator1: type fixed, parent base_link, child rotator_link1, origin xyz=0 0.04 0.021352, axis 0 0 1
- added joint rotator2: type continuous, parent base_link, child rotator_link2, origin xyz=0.026 -0.030397 0.021352 rpy=0 0 0.1185, axis 0 0 1, limit lower=-1.57 upper=1.57 effort=30 velocity=5
- added joint rotator3: type continuous, parent base_link, child rotator_link3, origin xyz=-0.026 -0.030397 0.021352 rpy=0 0 -0.1185, axis 0 0 1, limit lower=-1.57 upper=1.57 effort=30 velocity=5, mimic joint=rotator2 multiplier=-1

Commit message: Changed stl files to dae files to get textures in Rviz

File: wezelROS/description/urdf/gripper.urdf (robot description, URDF)
Before this commit: robot gripper, 7 links, 6 joints
Links:
- link base_link: geometry visual mesh filename=package://wezelROS/description/meshes/base.dae
- link finger_link1: geometry visual mesh filename=package://wezelROS/description/meshes/finger.dae
- link finger_link2: geometry visual mesh filename=package://wezelROS/description/meshes/finger.dae
- link finger_link3: geometry visual mesh filename=package://wezelROS/description/meshes/finger.dae
- link rotator_link1: geometry visual mesh filename=package://wezelROS/description/meshes/finger_rotator.dae
- link rotator_link2: geometry visual mesh filename=package://wezelROS/description/meshes/finger_rotator.dae
- link rotator_link3: geometry visual mesh filename=package://wezelROS/description/meshes/finger_rotator.dae

Commit message: Added collision and inertial tags

File: wezelROS/description/urdf/gripper.urdf (robot description, URDF)
Before this commit: robot gripper, 7 links, 6 joints
Links:
- link base_link: mass None -> 0.848; geometry collision mesh filename=package://wezelROS/description/meshes/base.dae; visual mesh filename=package://wezelROS/description/meshes/base.dae
- link finger_link1: mass None -> 0.025; geometry collision mesh filename=package://wezelROS/description/meshes/finger.dae; visual mesh filename=package://wezelROS/description/meshes/finger.dae
- link finger_link2: mass None -> 0.025; geometry collision mesh filename=package://wezelROS/description/meshes/finger.dae; visual mesh filename=package://wezelROS/description/meshes/finger.dae
- link finger_link3: mass None -> 0.025; geometry collision mesh filename=package://wezelROS/description/meshes/finger.dae; visual mesh filename=package://wezelROS/description/meshes/finger.dae
- link rotator_link1: mass None -> 0.011; geometry collision mesh filename=package://wezelROS/description/meshes/finger_rotator.dae; visual mesh filename=package://wezelROS/description/meshes/finger_rotator.dae
- link rotator_link2: mass None -> 0.011; geometry collision mesh filename=package://wezelROS/description/meshes/finger_rotator.dae; visual mesh filename=package://wezelROS/description/meshes/finger_rotator.dae
- link rotator_link3: mass None -> 0.011; geometry collision mesh filename=package://wezelROS/description/meshes/finger_rotator.dae; visual mesh filename=package://wezelROS/description/meshes/finger_rotator.dae
